File: hardware/f411_dev_board/f411_dev_board.kicad_sch (KiCad schematic)
At the start: 18 parts, among them U1 STM32F411CEU6, Y1 24MHz

Commit message: more pcb
Parts:
- added C11: 10u, Capacitor_SMD:C_0603_1608Metric, symbol Device:C_Small
- added C12: 22u, Capacitor_SMD:C_0603_1608Metric, symbol Device:C_Small
- added D1: LED_GREEN, LED_SMD:LED_0402_1005Metric, symbol Device:LED_Small
- added D2: LED_RED, LED_SMD:LED_0402_1005Metric, symbol Device:LED_Small
- added J1, J2: Conn_01x15, Connector_PinHeader_2.54mm:PinHeader_1x15_P2.54mm_Vertical, symbol Connector_Generic:Conn_01x15
- added J3: USB_C_Receptacle_USB2.0_14P, Connector_USB:USB_C_Receptacle_GCT_USB4105-xx-A_16P_TopMnt_Horizontal, symbol Connector:USB_C_Receptacle_USB2.0_14P
- added R1, R2, R7: 5.1k, Resistor_SMD:R_0402_1005Metric, symbol Device:R_Small
- added R6: 1k, Resistor_SMD:R_0402_1005Metric, symbol Device:R_Small
- added SW1: SW_SPDT, symbol Switch:SW_SPDT
- added U2: USBLC6-2SC6, Package_TO_SOT_SMD:SOT-23-6, symbol Power_Protection:USBLC6-2SC6
- added U3: AMS1117-3.3, Package_TO_SOT_SMD:SOT-223-3_TabPin2, symbol Regulator_Linear:AMS1117-3.3
- C1, C10, C2, C3, C4, C6: footprint (none) -> Capacitor_SMD:C_0402_1005Metric
- C13: renamed from C11; footprint (none) -> Capacitor_SMD:C_0402_1005Metric
- C14: renamed from C12; footprint (none) -> Capacitor_SMD:C_0402_1005Metric
- C5, C7, C8, C9: footprint (none) -> Capacitor_SMD:C_0603_1608Metric
- R3: renamed from R2; footprint (none) -> Resistor_SMD:R_0402_1005Metric
- R4: renamed from R1; footprint (none) -> Resistor_SMD:R_0402_1005Metric
- R5: renamed from R3; footprint (none) -> Resistor_SMD:R_0402_1005Metric
Connections:
- net +3V3: now also C12.1, D2.2 (A), J1.15 (Pin_15), J2.3 (Pin_3), R6.2, SW1.1 (A), U3.2 (VO)
- net BOOT0: now also R4.2; no longer R4.1
- net GND: now also C11.2, C12.2, J1.14 (Pin_14), J2.2 (Pin_2), J3.A1 (GND), J3.A12 (GND), J3.B1 (GND), J3.B12 (GND), R1.2, R2.2, R7.2, SW1.3 (C), U2.2 (GND), U3.1 (GND); no longer R4.2
- net PA0: now reaches U1.10 (PA0)
- net PA0: now also J2.4 (Pin_4)
- net PA1: now reaches U1.11 (PA1)
- net PA1: now also J2.5 (Pin_5)
- net PA2: now reaches U1.12 (PA2)
- net PA2: now also J2.6 (Pin_6)
- net PA3: now reaches U1.13 (PA3)
- net PA3: now also J2.7 (Pin_7)
- net PA4: now reaches U1.14 (PA4)
- net PA4: now also J2.8 (Pin_8)
- net PA5: now reaches U1.15 (PA5)
- net PA5: now also J2.9 (Pin_9)
- net PA6: now reaches U1.16 (PA6)
- net PA6: now also J2.10 (Pin_10)
- net PA7: now reaches U1.17 (PA7)
- net PA7: now also J2.11 (Pin_11)
- net PB0: now reaches U1.18 (PB0)
- net PB0: now also J1.1 (Pin_1)
- net PB1: now reaches U1.19 (PB1)
- net PB1: now also J1.2 (Pin_2)
- net BUILTIN_LED: now reaches U1.2 (PC13)
- net BUILTIN_LED: now also D1.1 (K)
- net PB2: now reaches U1.20 (PB2)
- net PB2: now also J1.3 (Pin_3)
- net PB10: now reaches U1.21 (PB10)
- net PB10: now also J1.11 (Pin_11)
- net PB12: now reaches U1.25 (PB12)
- net PB12: now also J1.12 (Pin_12)
- net PA8: now reaches U1.29 (PA8)
- net PA8: now also J2.12 (Pin_12)
- net PA9: now reaches U1.30 (PA9)
- net PA9: now also J2.13 (Pin_13)
- net PA10: now reaches U1.31 (PA10)
- net PA10: now also J2.14 (Pin_14)
- net USB_D-: now reaches U1.32 (PA11)
- net USB_D-: now also U2.6 (I/O1)
- net USB_D+: now reaches U1.33 (PA12)
- net USB_D+: now also U2.4 (I/O2)
- net PA13: now reaches U1.34 (PA13)
- net PA13: now also J2.15 (Pin_15)
- net PB3: now reaches U1.39 (PB3)
- net PB3: now also J1.4 (Pin_4)
- net PB4: now reaches U1.40 (PB4)
- net PB4: now also J1.5 (Pin_5)
- net PB5: now reaches U1.41 (PB5)
- net PB5: now also J1.6 (Pin_6)
- net PB6: now reaches U1.42 (PB6)
- net PB6: now also J1.7 (Pin_7)
- net PB7: now reaches U1.43 (PB7)
- net PB7: now also J1.8 (Pin_8)
- net PB8: now reaches U1.45 (PB8)
- net PB8: now also J1.9 (Pin_9)
- net PB9: now reaches U1.46 (PB9)
- net PB9: now also J1.10 (Pin_10)
- new net: J3.A5 (CC1), R1.1
- new net: J3.B5 (CC2), R2.1
- new net: R4.1, SW1.2 (B)
- new net BUILTIN_LED_A: D1.2 (A), R6.1
- new net PWR_LED_K: D2.1 (K), R7.1
- new net USB_CONN_D+: J3.A6 (D+), J3.B6 (D+), U2.3 (I/O2)
- new net USB_CONN_D-: J3.A7 (D-), J3.B7 (D-), U2.1 (I/O1)
- new net VBUS: C11.1, J1.13 (Pin_13), J2.1 (Pin_1), J3.A4 (VBUS), J3.A9 (VBUS), J3.B4 (VBUS), J3.B9 (VBUS), U2.5 (VBUS), U3.3 (VI)
- no-connect marks 0 -> 8
Other:
- moved on the sheet: C13, C14, R4, R5, U1, Y1

Commit message: more pcb again
Parts:
- removed J3: USB_C_Receptacle_USB2.0_14P, Connector_USB:USB_C_Receptacle_GCT_USB4105-xx-A_16P_TopMnt_Horizontal, symbol Connector:USB_C_Receptacle_USB2.0_14P
- removed R5: 0R, Resistor_SMD:R_0402_1005Metric, symbol Device:R_Small
- added J3: Conn_01x04, Connector_PinHeader_2.54mm:PinHeader_1x04_P2.54mm_Horizontal, symbol Connector_Generic:Conn_01x04
- added J4: USB_C_Receptacle_USB2.0_16P, Connector_USB:USB_C_Receptacle_GCT_USB4105-xx-A_16P_TopMnt_Horizontal, symbol Connector:USB_C_Receptacle_USB2.0_16P
- added SW2: SW_Push, Button_Switch_SMD:SW_Push_1P1T_XKB_TS-1187A, symbol Switch:SW_Push
- FB1: footprint (none) -> Inductor_SMD:L_0603_1608Metric
- SW1: footprint (none) -> Button_Switch_THT:SW_Slide_SPDT_Straight_CK_OS102011MS2Q
- Y1: footprint (none) -> Crystal:Crystal_SMD_3225-4Pin_3.2x2.5mm
Connections:
- net +3V3: now also J3.4 (Pin_4)
- net GND: now also J3.2 (Pin_2), J4.A1 (GND), J4.A12 (GND), J4.B1 (GND), J4.B12 (GND), SW2.1
- net HSE_OUT: now also C14.1, Y1.3
- net PA0: now also J1.1 (Pin_1); no longer J2.4 (Pin_4)
- net PA1: now also J1.2 (Pin_2); no longer J2.5 (Pin_5)
- net PA2: now also J1.3 (Pin_3); no longer J2.6 (Pin_6)
- net PA3: now also J1.4 (Pin_4); no longer J2.7 (Pin_7)
- net PA4: now also J1.5 (Pin_5); no longer J2.8 (Pin_8)
- net PA5: now also J1.6 (Pin_6); no longer J2.9 (Pin_9)
- net PA6: now also J1.7 (Pin_7); no longer J2.10 (Pin_10)
- net PA7: now also J1.8 (Pin_8); no longer J2.11 (Pin_11)
- net PB0: now also J1.9 (Pin_9); no longer J1.1 (Pin_1)
- net PB1: now also J1.10 (Pin_10); no longer J1.2 (Pin_2)
- net PB10: now also J1.12 (Pin_12); no longer J1.11 (Pin_11)
- net PB12: now also J2.15 (Pin_15); no longer J1.12 (Pin_12)
- net PB2: now also J1.11 (Pin_11); no longer J1.3 (Pin_3)
- net PB3: now also J2.10 (Pin_10); no longer J1.4 (Pin_4)
- net PB4: now also J2.9 (Pin_9); no longer J1.5 (Pin_5)
- net PB5: now also J2.8 (Pin_8); no longer J1.6 (Pin_6)
- net PB6: now also J2.7 (Pin_7); no longer J1.7 (Pin_7)
- net PB7: now also J2.6 (Pin_6); no longer J1.8 (Pin_8)
- net PB8: now also J2.5 (Pin_5); no longer J1.9 (Pin_9)
- net PB9: now also J2.4 (Pin_4); no longer J1.10 (Pin_10)
- net RESET: now also SW2.2
- net USB_CONN_D+: now also J4.A6 (D+), J4.B6 (D+)
- net USB_CONN_D-: now also J4.A7 (D-), J4.B7 (D-)
- net VBUS: now also J4.A4 (VBUS), J4.A9 (VBUS), J4.B4 (VBUS), J4.B9 (VBUS)
- net CC1: now reaches R1.1
- net CC1: now also J4.A5 (CC1)
- net CC2: now reaches R2.1
- net CC2: now also J4.B5 (CC2)
- net BOOT0_SW: now reaches R4.1, SW1.2 (B)
- net SWCLK: now reaches U1.37 (PA14)
- net SWCLK: now also J3.3 (Pin_3)
- net PA15: now reaches U1.38 (PA15)
- net PA15: now also J2.11 (Pin_11)
- net PA13 renamed SWDIO
- net SWDIO: now also J3.1 (Pin_1); no longer J2.15 (Pin_15)
Other:
- moved on the sheet: C10, C9, R1, R2, R3, R4, SW1
