File: hardware/f411_dev_board/f411_dev_board.kicad_sch (KiCad schematic)
At the start: 33 parts, among them J1 Conn_01x15, J2 Conn_01x15, J3 Conn_01x04, J4 USB_C_Receptacle_USB2.0_16P, SW1 SW_SPDT, SW2 SW_Push, U1 STM32F411CEU6, U2 USBLC6-2SC6, U3 AMS1117-3.3, Y1 24MHz

Commit message: finish pcb v2
also reorganized schematic
Parts:
- SW1: value SW_SPDT -> SW_BOOT0
- SW2: value SW_Push -> SW_RESET
Connections:
- net GND: now also J4.SH (SHIELD)
- net PA10: now also J2.15 (Pin_15); no longer J2.14 (Pin_14)
- net PA8: now also J2.13 (Pin_13); no longer J2.12 (Pin_12)
- net PA9: now also J2.14 (Pin_14); no longer J2.13 (Pin_13)
- net PB12: now also J2.12 (Pin_12); no longer J2.15 (Pin_15)
- no-connect marks 8 -> 7
Other:
- note added: "24MHz Crystal"
- note added: "BOOT0"
- note added: "Decoupling Caps"
- note added: "ESD"
- note added: "GPIO Headers"
- note added: "LDO"
- note added: "POWER LED"
- note added: "RESET"
- note added: "STM32F411CEU6"
- note added: "Serial Wire Header"
- note added: "USB-C"
- note added: "USER LED"
- moved on the sheet: C1, C10, C11, C12, C13, C14, C2, C3, C4, C5, C6, C7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
